Commit message: Rotating base to align with x axis

File: rsk_urdf/robot.urdf (robot description, URDF)
Before this commit: robot rsk_urdf, 114 links, 113 joints
Joints:
- joint base_18650_2_fixed: origin xyz=-0.0570303 0.00914608 0.0556537 rpy=-3.14159 6.23961e-54 1.0472 -> xyz=-0.00915859 -0.0570304 0.0732537 rpy=-3.14159 6.23961e-54 2.61799
- joint base_18650_fixed: origin xyz=-0.0400271 0.0225965 0.0556537 rpy=-3.14159 1.87188e-53 1.0472 -> xyz=-0.022609 -0.0400272 0.0732537 rpy=-3.14159 1.87188e-53 2.61799
- joint base_blue1_blue_fixed: origin xyz=0.00122945 -0.000286033 0.0505 rpy=-2.85456e-24 2.48154e-24 -4.996e-16 -> xyz=0.000273519 0.00122933 0.0681 rpy=-2.85456e-24 2.48154e-24 1.5708
- joint base_blue1_white_fixed: origin xyz=4.19044e-16 -2.22673e-06 0.0653 rpy=-3.14159 -2.48154e-24 3.14159 -> xyz=-1.02871e-05 -1.23093e-07 0.0829 rpy=-3.14159 -2.48154e-24 -1.5708
- joint base_board_fixed: origin xyz=0 0 0 rpy=0 -0 0 -> xyz=-1.25138e-05 -1.23093e-07 0.0176 rpy=0 -0 1.5708
- joint base_coil_fixed: origin xyz=-0.0066 -0.0695 8.67362e-19 rpy=-1.5708 -1.5708 0 -> xyz=0.0694875 -0.00660012 0.0176 rpy=-0 -1.5708 0
- joint base_coupler_fixed: origin xyz=0.0156562 -0.0329573 0.0335 rpy=1.6719e-54 6.23961e-54 1.0472 -> xyz=0.0329448 0.015656 0.0511 rpy=1.6719e-54 6.23961e-54 2.61799
- joint base_frame_2_fixed: origin xyz=-0.0066 -0.0695 0 rpy=-1.5708 -1.5708 0 -> xyz=0.0694875 -0.00660012 0.0176 rpy=-0 -1.5708 0
- joint base_frame_fixed: origin xyz=-1.04083e-17 8.32667e-17 0.0305 rpy=-6.5253e-55 6.5253e-55 -4.996e-16 -> xyz=-1.25138e-05 -1.23093e-07 0.0481 rpy=-6.5253e-55 6.5253e-55 1.5708
- joint base_hex_socket_head_cap_screw_m3x0_50_x_25_x_18__e477b94a6da3e3efbf1606183756b785_2_fixed: origin xyz=0.00975 0.0331 -0.0046 rpy=3.14159 -0 0 -> xyz=-0.0331125 0.00974988 0.013 rpy=3.14159 -0 1.5708
- joint base_hex_socket_head_cap_screw_m3x0_50_x_25_x_18__e477b94a6da3e3efbf1606183756b785_3_fixed: origin xyz=0.0237904 -0.0249937 -0.0046 rpy=3.14159 -0 0 -> xyz=0.0249812 0.0237903 0.013 rpy=3.14159 -0 1.5708
- joint base_hex_socket_head_cap_screw_m3x0_50_x_25_x_18__e477b94a6da3e3efbf1606183756b785_4_fixed: origin xyz=0.0335404 -0.00810625 -0.0046 rpy=3.14159 -0 0 -> xyz=0.00809374 0.0335403 0.013 rpy=3.14159 -0 1.5708
- joint base_hex_socket_head_cap_screw_m3x0_50_x_25_x_18__e477b94a6da3e3efbf1606183756b785_5_fixed: origin xyz=-0.0237904 -0.0249937 -0.0046 rpy=3.14159 -0 0 -> xyz=0.0249812 -0.0237906 0.013 rpy=3.14159 -0 1.5708
- joint base_hex_socket_head_cap_screw_m3x0_50_x_25_x_18__e477b94a6da3e3efbf1606183756b785_6_fixed: origin xyz=-0.00975 0.0331 -0.0046 rpy=3.14159 -0 0 -> xyz=-0.0331125 -0.00975012 0.013 rpy=3.14159 -0 1.5708
- joint base_hex_socket_head_cap_screw_m3x0_50_x_25_x_18__e477b94a6da3e3efbf1606183756b785_fixed: origin xyz=-0.0335404 -0.00810625 -0.0046 rpy=3.14159 -0 0 -> xyz=0.00809374 -0.0335406 0.013 rpy=3.14159 -0 1.5708
- joint base_hex_socket_head_cap_screw_m3x0_50_x_6__acf8a907a0472c0ae6086bf20401fa07_2_fixed: origin xyz=0 -0.0475 -0.0046 rpy=3.14159 -0 0 -> xyz=0.0474875 -1.23093e-07 0.013 rpy=3.14159 -0 1.5708
- joint base_hex_socket_head_cap_screw_m3x0_50_x_6__acf8a907a0472c0ae6086bf20401fa07_fixed: origin xyz=0 -0.062 -0.0046 rpy=3.14159 -0 0 -> xyz=0.0619875 -1.23093e-07 0.013 rpy=3.14159 -0 1.5708
- joint base_m3_spacer__length_0_006_meter_2_fixed: origin xyz=-0.0335404 -0.00810625 0.0245 rpy=0 -0 0.523599 -> xyz=0.00809374 -0.0335406 0.0421 rpy=0 -0 2.0944
- joint base_m3_spacer__length_0_006_meter_3_fixed: origin xyz=0.0237904 -0.0249937 0.0245 rpy=0 -0 2.61799 -> xyz=0.0249812 0.0237903 0.0421 rpy=0 -0 -2.0944
- joint base_m3_spacer__length_0_006_meter_4_fixed: origin xyz=0.00975 0.0331 0.0245 rpy=0 -0 -1.5708 -> xyz=-0.0331125 0.00974988 0.0421 rpy=0 -0 -4.996e-16
- joint base_m3_spacer__length_0_006_meter_5_fixed: origin xyz=0.0335404 -0.00810625 0.0245 rpy=0 -0 2.61799 -> xyz=0.00809374 0.0335403 0.0421 rpy=0 -0 -2.0944
- joint base_m3_spacer__length_0_006_meter_6_fixed: origin xyz=-0.00975 0.0331 0.0245 rpy=0 -0 -1.5708 -> xyz=-0.0331125 -0.00975012 0.0421 rpy=0 -0 -4.996e-16
- joint base_m3_spacer__length_0_006_meter_fixed: origin xyz=-0.0237904 -0.0249937 0.0245 rpy=0 -0 0.523599 -> xyz=0.0249812 -0.0237906 0.0421 rpy=0 -0 2.0944
- joint base_m3_spacer__length_0_02_meter_2_fixed: origin xyz=0.0335404 -0.00810625 0.0335 rpy=-5.70911e-24 -3.26265e-55 -4.996e-16 -> xyz=0.00809374 0.0335403 0.0511 rpy=-5.70911e-24 -3.26265e-55 1.5708
- joint base_m3_spacer__length_0_02_meter_3_fixed: origin xyz=-0.00975 0.0331 0.0335 rpy=-5.70911e-24 -3.26265e-55 -4.996e-16 -> xyz=-0.0331125 -0.00975012 0.0511 rpy=-5.70911e-24 -3.26265e-55 1.5708
- joint base_m3_spacer__length_0_02_meter_4_fixed: origin xyz=0.0237904 -0.0249937 0.0335 rpy=-5.70911e-24 -3.26265e-55 -4.996e-16 -> xyz=0.0249812 0.0237903 0.0511 rpy=-5.70911e-24 -3.26265e-55 1.5708
- joint base_m3_spacer__length_0_02_meter_5_fixed: origin xyz=0.00975 0.0331 0.0335 rpy=-5.70911e-24 -3.26265e-55 -4.996e-16 -> xyz=-0.0331125 0.00974988 0.0511 rpy=-5.70911e-24 -3.26265e-55 1.5708
- joint base_m3_spacer__length_0_02_meter_6_fixed: origin xyz=-0.0335404 -0.00810625 0.0335 rpy=-5.70911e-24 -3.26265e-55 -4.996e-16 -> xyz=0.00809374 -0.0335406 0.0511 rpy=-5.70911e-24 -3.26265e-55 1.5708
- joint base_m3_spacer__length_0_02_meter_fixed: origin xyz=-0.0237904 -0.0249937 0.0335 rpy=-5.70911e-24 -3.26265e-55 -4.996e-16 -> xyz=0.0249812 -0.0237906 0.0511 rpy=-5.70911e-24 -3.26265e-55 1.5708
- joint base_m3_spacer__length_0_03_meter_10_fixed: origin xyz=0.0695237 0.0135814 0 rpy=0 -0 0 -> xyz=-0.0135939 0.0695236 0.0176 rpy=0 -0 1.5708
- joint base_m3_spacer__length_0_03_meter_2_fixed: origin xyz=-0.0792917 -0.00733717 0 rpy=0 -0 0 -> xyz=0.00732465 -0.0792918 0.0176 rpy=0 -0 1.5708
- joint base_m3_spacer__length_0_03_meter_3_fixed: origin xyz=0.0465237 0.0534186 0 rpy=0 -0 0 -> xyz=-0.0534311 0.0465236 0.0176 rpy=0 -0 1.5708
- joint base_m3_spacer__length_0_03_meter_4_fixed: origin xyz=0.046 -0.065 0 rpy=0 -0 0 -> xyz=0.0649875 0.0459999 0.0176 rpy=0 -0 1.5708
- joint base_m3_spacer__length_0_03_meter_5_fixed: origin xyz=-0.0695237 0.0135814 0 rpy=0 -0 0 -> xyz=-0.0135939 -0.0695238 0.0176 rpy=0 -0 1.5708
- joint base_m3_spacer__length_0_03_meter_6_fixed: origin xyz=-0.0332917 0.0723372 0 rpy=0 -0 0 -> xyz=-0.0723497 -0.0332918 0.0176 rpy=0 -0 1.5708
- joint base_m3_spacer__length_0_03_meter_7_fixed: origin xyz=-0.0465237 0.0534186 0 rpy=0 -0 0 -> xyz=-0.0534311 -0.0465238 0.0176 rpy=0 -0 1.5708
- joint base_m3_spacer__length_0_03_meter_8_fixed: origin xyz=-0.046 -0.065 0 rpy=0 -0 0 -> xyz=0.0649875 -0.0460001 0.0176 rpy=0 -0 1.5708
- joint base_m3_spacer__length_0_03_meter_9_fixed: origin xyz=0.0792917 -0.00733717 0 rpy=0 -0 0 -> xyz=0.00732465 0.0792915 0.0176 rpy=0 -0 1.5708
- joint base_m3_spacer__length_0_03_meter_fixed: origin xyz=0.0332917 0.0723372 0 rpy=0 -0 0 -> xyz=-0.0723497 0.0332915 0.0176 rpy=0 -0 1.5708
- joint base_marker_fixed: origin xyz=4.33681e-16 1.60982e-15 0.0505 rpy=-5.70911e-24 -3.26265e-55 -4.996e-16 -> xyz=-1.25138e-05 -1.23093e-07 0.0681 rpy=-5.70911e-24 -3.26265e-55 1.5708
- joint base_motorbox_bottom_2_fixed: origin xyz=-0.011376 -0.0134962 0.012 rpy=0 -0 2.0944 -> xyz=0.0134836 -0.0113761 0.0296 rpy=0 -0 -2.61799
- joint base_motorbox_bottom_3_fixed: origin xyz=0.017376 -0.00310385 0.012 rpy=0 -0 -2.0944 -> xyz=0.00309133 0.0173759 0.0296 rpy=0 -0 -0.523599
- joint base_motorbox_bottom_fixed: origin xyz=-0.006 0.0166 0.012 rpy=0 -0 -1.7792e-16 -> xyz=-0.0166125 -0.00600012 0.0296 rpy=0 -0 1.5708
- joint base_motorbox_top_2_fixed: origin xyz=-0.011376 -0.0134962 0.012 rpy=0 -0 2.0944 -> xyz=0.0134836 -0.0113761 0.0296 rpy=0 -0 -2.61799
- joint base_motorbox_top_3_fixed: origin xyz=0.017376 -0.00310385 0.012 rpy=0 -0 -2.0944 -> xyz=0.00309133 0.0173759 0.0296 rpy=0 -0 -0.523599
- joint base_motorbox_top_fixed: origin xyz=-0.006 0.0166 0.012 rpy=0 -0 -5.27356e-16 -> xyz=-0.0166125 -0.00600012 0.0296 rpy=0 -0 1.5708
- joint base_n20_2_fixed: origin xyz=-0.011376 -0.0134962 0.012 rpy=0 -0 2.0944 -> xyz=0.0134836 -0.0113761 0.0296 rpy=0 -0 -2.61799
- joint base_n20_3_fixed: origin xyz=0.017376 -0.00310385 0.012 rpy=0 -0 -2.0944 -> xyz=0.00309133 0.0173759 0.0296 rpy=0 -0 -0.523599
- joint base_n20_fixed: origin xyz=-0.006 0.0166 0.012 rpy=0 -0 -1.66533e-16 -> xyz=-0.0166125 -0.00600012 0.0296 rpy=0 -0 1.5708
- joint kicker: origin xyz=-1.73472e-18 -0.0405 0.00775 rpy=-1.5708 -1.5708 0 -> xyz=0.0404875 -1.23093e-07 0.02535 rpy=-0 -1.5708 0
- joint wheel1_passive_10: origin xyz=1.73472e-18 -0.0285 -0.01 rpy=1.5708 -4.78251e-18 1.5708 -> xyz=1.73472e-18 -0.0285 -0.01 rpy=1.5708 -3.8774e-18 1.5708
- joint wheel1_passive_13: origin xyz=0.023057 -0.0167519 -0.01 rpy=1.5708 7.01929e-15 -0.628319 -> xyz=0.023057 -0.0167519 -0.01 rpy=1.5708 7.03424e-15 -0.628319
- joint wheel1_passive_14: origin xyz=0.0271051 -0.00880698 -0.01 rpy=1.5708 7.51136e-15 -0.314159 -> xyz=0.0271051 -0.00880698 -0.01 rpy=1.5708 7.48324e-15 -0.314159
- joint wheel1_passive_15: origin xyz=0.0285 -1.73472e-17 -0.01 rpy=1.5708 -2.63053e-14 -3.93956e-16 -> xyz=0.0285 -1.38778e-17 -0.01 rpy=1.5708 -2.63408e-14 -4.02599e-16
- joint wheel1_passive_16: origin xyz=0.0271051 0.00880698 -0.01 rpy=1.5708 2.27736e-17 -2.82743 -> xyz=0.0271051 0.00880698 -0.01 rpy=1.5708 4.63079e-18 -2.82743
- joint wheel1_passive_17: origin xyz=0.023057 0.0167519 -0.01 rpy=1.5708 4.17525e-17 -2.51327 -> xyz=0.023057 0.0167519 -0.01 rpy=1.5708 6.01992e-17 -2.51327
- joint wheel1_passive_18: origin xyz=0.0167519 0.023057 -0.01 rpy=1.5708 1.79434e-17 -2.19911 -> xyz=0.0167519 0.023057 -0.01 rpy=1.5708 4.91315e-17 -2.19911
- joint wheel1_passive_2: origin xyz=-0.0167519 0.023057 -0.01 rpy=-1.5708 3.18404e-16 -0.942478 -> xyz=-0.0167519 0.023057 -0.01 rpy=-1.5708 2.93259e-16 -0.942478
- joint wheel1_passive_20: origin xyz=2.1684e-17 0.0285 -0.01 rpy=8.13793e-17 -1.5708 0 -> xyz=1.73472e-17 0.0285 -0.01 rpy=7.27361e-17 -1.5708 0
- joint wheel1_passive_3: origin xyz=-0.023057 0.0167519 -0.01 rpy=1.5708 -8.6135e-17 -0.628319 -> xyz=-0.023057 0.0167519 -0.01 rpy=1.5708 -3.90162e-17 -0.628319
- joint wheel1_passive_4: origin xyz=-0.0271051 0.00880698 -0.01 rpy=1.5708 -3.9118e-14 -0.314159 -> xyz=-0.0271051 0.00880698 -0.01 rpy=1.5708 -3.91234e-14 -0.314159
- joint wheel1_passive_5: origin xyz=-0.0285 -1.38778e-17 -0.01 rpy=1.5708 -6.94375e-14 -3.52311e-16 -> xyz=-0.0285 0 -0.01 rpy=1.5708 -6.94415e-14 -3.05443e-16
- joint wheel1_passive_6: origin xyz=-0.0271051 -0.00880698 -0.01 rpy=1.5708 -7.82847e-17 0.314159 -> xyz=-0.0271051 -0.00880698 -0.01 rpy=1.5708 -5.27049e-17 0.314159
- joint wheel1_passive_7: origin xyz=-0.023057 -0.0167519 -0.01 rpy=1.5708 -1.36975e-14 0.628319 -> xyz=-0.023057 -0.0167519 -0.01 rpy=1.5708 -1.36878e-14 0.628319
- joint wheel1_passive_8: origin xyz=-0.0167519 -0.023057 -0.01 rpy=1.5708 -1.76654e-15 0.942478 -> xyz=-0.0167519 -0.023057 -0.01 rpy=1.5708 -1.74069e-15 0.942478
- joint wheel1_speed: origin xyz=0.0408764 -0.0236 0.017 rpy=1.5708 -0.355266 -2.0944 -> xyz=0.0235875 0.0408763 0.0346 rpy=1.5708 -0.355266 -0.523599
- joint wheel2_passive1: origin xyz=0.0271051 -0.00880698 -0.01 rpy=-1.5708 -2.20675e-14 -0.314159 -> xyz=0.0271051 -0.00880698 -0.01 rpy=-1.5708 -2.20929e-14 -0.314159
- joint wheel2_passive11: origin xyz=0.00880698 0.0271051 -0.01 rpy=1.5708 1.28548e-16 -1.88496 -> xyz=0.00880698 0.0271051 -0.01 rpy=1.5708 1.32683e-16 -1.88496
- joint wheel2_passive12: origin xyz=1.8894e-18 0.0285 -0.01 rpy=-3.14159 1.5708 0 -> xyz=-3.75574e-18 0.0285 -0.01 rpy=-3.14159 1.5708 0
- joint wheel2_passive17: origin xyz=-0.023057 -0.0167519 -0.01 rpy=1.5708 3.5412e-17 0.628319 -> xyz=-0.023057 -0.0167519 -0.01 rpy=1.5708 3.60754e-18 0.628319
- joint wheel2_passive19: origin xyz=-0.0285 0 -0.01 rpy=-1.5708 1.5708 0 -> xyz=-0.0285 -6.93889e-18 -0.01 rpy=-1.5708 1.5708 0
- joint wheel2_passive3: origin xyz=0.0167519 -0.023057 -0.01 rpy=-1.5708 -9.8851e-15 2.19911 -> xyz=0.0167519 -0.023057 -0.01 rpy=-1.5708 -9.83757e-15 2.19911
- joint wheel2_passive5: origin xyz=-5.01677e-18 -0.0285 -0.01 rpy=-1.66533e-16 -1.5708 0 -> xyz=-6.4798e-18 -0.0285 -0.01 rpy=-1.66533e-16 -1.5708 0
- joint wheel2_passive7: origin xyz=0.0285 -3.46945e-18 -0.01 rpy=-1.5708 1.5708 0 -> xyz=0.0285 -1.38778e-17 -0.01 rpy=-1.5708 1.5708 0
- joint wheel2_speed: origin xyz=-0.0408764 -0.0236 0.017 rpy=-1.5708 -1.08703e-13 -1.0472 -> xyz=0.0235875 -0.0408765 0.0346 rpy=-1.5708 -1.08703e-13 0.523599
- joint wheel3_passive1: origin xyz=1.32815e-17 0.0285 -0.01 rpy=3.14159 -1.5708 0 -> xyz=1.2902e-17 0.0285 -0.01 rpy=3.14159 -1.5708 0
- joint wheel3_passive11: origin xyz=1.01915e-17 -0.0285 -0.01 rpy=3.14159 -1.5708 0 -> xyz=1.06252e-17 -0.0285 -0.01 rpy=3.14159 -1.5708 0
- joint wheel3_passive6: origin xyz=-0.0285 0 -0.01 rpy=1.5708 -7.5361e-16 -9.43428e-17 -> xyz=-0.0285 6.93889e-18 -0.01 rpy=1.5708 -7.5361e-16 -9.43428e-17
- joint wheel3_speed: origin xyz=-1.92398e-17 0.0472 0.017 rpy=1.5708 0.0233987 -1.66533e-16 -> xyz=-0.0472125 -1.23093e-07 0.0346 rpy=1.5708 0.0233987 1.5708
