Commit message: Update config, README and add momo_ mujoco

File: momo_urdf/robot.urdf (robot description, URDF)
Before this commit: robot momo, 60 links, 59 joints
Links:
- removed link logitech_back
- removed link logitech_front
- removed link logitech_left
- removed link logitech_right
- removed link realsense_back
- removed link realsense_front
- removed link velodyne
- added link back_logitech_frame, mass 1e-9
- added link back_realsense_frame, mass 1e-9
- added link front_logitech_frame, mass 1e-9
- added link front_realsense_frame, mass 1e-9
- added link left_logitech_frame, mass 1e-9
- added link right_logitech_frame, mass 1e-9
- added link velodyne_frame, mass 1e-9
- link back_left_wheel: geometry visual mesh filename=package://assets/merged/back_left_wheel_visual.stl
- link back_right_wheel: geometry visual mesh filename=package://assets/merged/back_right_wheel_visual.stl
- link base_link: geometry collision box size=0.435 0.645 0.276; collision box size=0.745 0.44 0.225
- link front_left_wheel: geometry visual mesh filename=package://assets/merged/front_left_wheel_visual.stl
- link front_right_wheel: geometry visual mesh filename=package://assets/merged/front_right_wheel_visual.stl
- link roller: geometry collision sphere radius=0.014; collision sphere radius=0.014
- link roller_10: geometry collision sphere radius=0.014; collision sphere radius=0.014
- link roller_11: geometry collision sphere radius=0.014; collision sphere radius=0.014
- link roller_12: geometry collision sphere radius=0.014; collision sphere radius=0.014
- link roller_13: geometry collision sphere radius=0.014; collision sphere radius=0.014
- link roller_14: geometry collision sphere radius=0.014; collision sphere radius=0.014
- link roller_15: geometry collision sphere radius=0.014; collision sphere radius=0.014
- link roller_16: geometry collision sphere radius=0.014; collision sphere radius=0.014
- link roller_17: geometry collision sphere radius=0.014; collision sphere radius=0.014
- link roller_18: geometry collision sphere radius=0.014; collision sphere radius=0.014
- link roller_19: geometry collision sphere radius=0.014; collision sphere radius=0.014
- link roller_2: geometry collision sphere radius=0.014; collision sphere radius=0.014
- link roller_20: geometry collision sphere radius=0.014; collision sphere radius=0.014
- link roller_21: geometry collision sphere radius=0.014; collision sphere radius=0.014
- link roller_22: geometry collision sphere radius=0.014; collision sphere radius=0.014
- link roller_23: geometry collision sphere radius=0.014; collision sphere radius=0.014
- link roller_24: geometry collision sphere radius=0.014; collision sphere radius=0.014
- link roller_25: geometry collision sphere radius=0.014; collision sphere radius=0.014
- link roller_26: geometry collision sphere radius=0.014; collision sphere radius=0.014
- link roller_27: geometry collision sphere radius=0.014; collision sphere radius=0.014
- link roller_28: geometry collision sphere radius=0.014; collision sphere radius=0.014
- link roller_29: geometry collision sphere radius=0.014; collision sphere radius=0.014
- link roller_3: geometry collision sphere radius=0.014; collision sphere radius=0.014
- link roller_30: geometry collision sphere radius=0.014; collision sphere radius=0.014
- link roller_31: geometry collision sphere radius=0.014; collision sphere radius=0.014
- link roller_32: geometry collision sphere radius=0.014; collision sphere radius=0.014
- link roller_33: geometry collision sphere radius=0.014; collision sphere radius=0.014
- link roller_34: geometry collision sphere radius=0.014; collision sphere radius=0.014
- link roller_35: geometry collision sphere radius=0.014; collision sphere radius=0.014
- link roller_36: geometry collision sphere radius=0.014; collision sphere radius=0.014
- link roller_37: geometry collision sphere radius=0.014; collision sphere radius=0.014
- link roller_38: geometry collision sphere radius=0.014; collision sphere radius=0.014
- link roller_39: geometry collision sphere radius=0.014; collision sphere radius=0.014
- link roller_4: geometry collision sphere radius=0.014; collision sphere radius=0.014
- link roller_40: geometry collision sphere radius=0.014; collision sphere radius=0.014
- link roller_41: geometry collision sphere radius=0.014; collision sphere radius=0.014
- link roller_42: geometry collision sphere radius=0.014; collision sphere radius=0.014
- link roller_43: geometry collision sphere radius=0.014; collision sphere radius=0.014
- link roller_44: geometry collision sphere radius=0.014; collision sphere radius=0.014
- link roller_45: geometry collision sphere radius=0.014; collision sphere radius=0.014
- link roller_46: geometry collision sphere radius=0.014; collision sphere radius=0.014
- link roller_47: geometry collision sphere radius=0.014; collision sphere radius=0.014
- link roller_48: geometry collision sphere radius=0.014; collision sphere radius=0.014
- link roller_5: geometry collision sphere radius=0.014; collision sphere radius=0.014
- link roller_6: geometry collision sphere radius=0.014; collision sphere radius=0.014
- link roller_7: geometry collision sphere radius=0.014; collision sphere radius=0.014
- link roller_8: geometry collision sphere radius=0.014; collision sphere radius=0.014
- link roller_9: geometry collision sphere radius=0.014; collision sphere radius=0.014
Joints:
- removed joint logitech_back_frame
- removed joint logitech_front_frame
- removed joint logitech_left_frame
- removed joint logitech_right_frame
- removed joint realsense_back_frame
- removed joint realsense_front_frame
- removed joint velodyne_frame
- added joint back_logitech_frame_frame: type fixed, parent base_link, child back_logitech_frame, origin xyz=-0.259083 1.41843e-05 0.408222 rpy=-1.5708 8.29069e-14 1.5708, axis 0 0 0
- added joint back_realsense_frame_frame: type fixed, parent base_link, child back_realsense_frame, origin xyz=-0.381177 0.000689294 0.31717 rpy=-1.5708 3.69437e-14 1.5708, axis 0 0 0
- added joint front_logitech_frame_frame: type fixed, parent base_link, child front_logitech_frame, origin xyz=0.150217 -1.41843e-05 0.408222 rpy=-1.5708 -3.69437e-14 -1.5708, axis 0 0 0
- added joint front_realsense_frame_frame: type fixed, parent base_link, child front_realsense_frame, origin xyz=0.272296 -0.00478981 0.31864 rpy=-1.5708 -3.69437e-14 -1.5708, axis 0 0 0
- added joint left_logitech_frame_frame: type fixed, parent base_link, child left_logitech_frame, origin xyz=-0.00691857 0.20665 0.408222 rpy=-1.5708 -3.31108e-15 -9.16481e-14, axis 0 0 0
- added joint right_logitech_frame_frame: type fixed, parent base_link, child right_logitech_frame, origin xyz=-0.00694694 -0.20665 0.408222 rpy=-1.5708 1.96259e-15 3.14159, axis 0 0 0
- added joint velodyne_frame_frame: type fixed, parent base_link, child velodyne_frame, origin xyz=-0.00693293 1.75362e-07 0.467529 rpy=1.66614e-14 4.87655e-14 -1.5708, axis 0 0 0
- joint back_left_wheel: axis 0 0 -1 -> 0 0 1; origin xyz=-0.2735 0.24 0.065 rpy=-1.5708 7.65429e-15 -3.14159 -> xyz=-0.2735 0.24 0.065 rpy=1.5708 7.65429e-15 -3.14159
- joint blw_r1: origin xyz=0.0299314 -0.0806297 -0.039 rpy=-0.747479 0.268603 2.20514 -> xyz=0.0299314 0.0806297 0.039 rpy=2.39411 -0.268603 -2.20514
- joint blw_r10: origin xyz=-0.080624 -0.0299395 -0.039 rpy=-0.747479 0.268603 0.634348 -> xyz=-0.080624 0.0299395 0.039 rpy=2.39411 -0.268603 -0.634348
- joint blw_r11: origin xyz=-0.0847889 0.0143821 -0.039 rpy=0.359043 0.714734 1.92274 -> xyz=-0.0847889 -0.0143821 0.039 rpy=-2.78255 -0.714734 -1.92274
- joint blw_r12: origin xyz=-0.066235 0.0548482 -0.039 rpy=0.359043 0.714734 1.39914 -> xyz=-0.066235 -0.0548482 0.039 rpy=-2.78255 -0.714734 -1.39914
- joint blw_r2: origin xyz=0.0662326 -0.054862 -0.039 rpy=-0.747479 0.268603 2.72874 -> xyz=0.0662326 0.054862 0.039 rpy=2.39411 -0.268603 -2.72874
- joint blw_r3: origin xyz=0.0847865 -0.0143959 -0.039 rpy=-0.359043 -0.714734 1.92274 -> xyz=0.0847865 0.0143959 0.039 rpy=2.78255 0.714734 -1.92274
- joint blw_r4: origin xyz=0.0806217 0.0299257 -0.039 rpy=-0.359043 -0.714734 2.44634 -> xyz=0.0806217 -0.0299257 0.039 rpy=2.78255 0.714734 -2.44634
- joint blw_r5: origin xyz=0.0548539 0.0662269 -0.039 rpy=-0.359043 -0.714734 2.96994 -> xyz=0.0548539 -0.0662269 0.039 rpy=2.78255 0.714734 -2.96994
- joint blw_r6: origin xyz=0.0143878 0.0847808 -0.039 rpy=-0.747479 0.268603 -1.46005 -> xyz=0.0143878 -0.0847808 0.039 rpy=2.39411 -0.268603 1.46005
- joint blw_r7: origin xyz=-0.0299338 0.0806159 -0.039 rpy=0.359043 0.714734 0.875544 -> xyz=-0.0299338 -0.0806159 0.039 rpy=-2.78255 -0.714734 -0.875544
- joint blw_r8: origin xyz=-0.0143902 -0.0847946 -0.039 rpy=-0.747479 0.268603 1.68155 -> xyz=-0.0143902 0.0847946 0.039 rpy=2.39411 -0.268603 -1.68155
- joint blw_r9: origin xyz=-0.0548563 -0.0662407 -0.039 rpy=-0.747479 0.268603 1.15795 -> xyz=-0.0548563 0.0662407 0.039 rpy=2.39411 -0.268603 -1.15795
- joint flw_r1: origin xyz=-0.014389 -0.0847877 -0.039 rpy=-0.359043 -0.714734 -2.78965 -> xyz=-0.014389 0.0847877 0.039 rpy=2.78255 0.714734 2.78965
- joint flw_r10: origin xyz=-0.0847877 0.014389 -0.039 rpy=-0.359043 -0.714734 1.92274 -> xyz=-0.0847877 -0.014389 0.039 rpy=2.78255 0.714734 -1.92274
- joint flw_r11: origin xyz=-0.0806228 -0.0299326 -0.039 rpy=-0.359043 -0.714734 2.44634 -> xyz=-0.0806228 0.0299326 0.039 rpy=2.78255 0.714734 -2.44634
- joint flw_r12: origin xyz=-0.0548551 -0.0662338 -0.039 rpy=-0.359043 -0.714734 2.96994 -> xyz=-0.0548551 0.0662338 0.039 rpy=2.78255 0.714734 -2.96994
- joint flw_r2: origin xyz=0.0299326 -0.0806228 -0.039 rpy=0.359043 0.714734 0.875544 -> xyz=0.0299326 0.0806228 0.039 rpy=-2.78255 -0.714734 -0.875544
- joint flw_r3: origin xyz=0.0662338 -0.0548551 -0.039 rpy=0.359043 0.714734 1.39914 -> xyz=0.0662338 0.0548551 0.039 rpy=-2.78255 -0.714734 -1.39914
- joint flw_r4: origin xyz=0.0847877 -0.014389 -0.039 rpy=0.359043 0.714734 1.92274 -> xyz=0.0847877 0.014389 0.039 rpy=-2.78255 -0.714734 -1.92274
- joint flw_r5: origin xyz=0.0806228 0.0299326 -0.039 rpy=-0.747479 0.268603 0.634348 -> xyz=0.0806228 -0.0299326 0.039 rpy=2.39411 -0.268603 -0.634348
- joint flw_r6: origin xyz=0.0548551 0.0662338 -0.039 rpy=-0.747479 0.268603 1.15795 -> xyz=0.0548551 -0.0662338 0.039 rpy=2.39411 -0.268603 -1.15795
- joint flw_r7: origin xyz=0.014389 0.0847877 -0.039 rpy=-0.747479 0.268603 1.68155 -> xyz=0.014389 -0.0847877 0.039 rpy=2.39411 -0.268603 -1.68155
- joint flw_r8: origin xyz=-0.0299326 0.0806228 -0.039 rpy=-0.747479 0.268603 2.20514 -> xyz=-0.0299326 -0.0806228 0.039 rpy=2.39411 -0.268603 -2.20514
- joint flw_r9: origin xyz=-0.0662338 0.0548551 -0.039 rpy=-0.747479 0.268603 2.72874 -> xyz=-0.0662338 -0.0548551 0.039 rpy=2.39411 -0.268603 -2.72874
- joint front_left_wheel: axis 0 0 -1 -> 0 0 1; origin xyz=0.2685 0.24 0.065 rpy=-1.5708 -6.32034e-16 -3.14159 -> xyz=0.2685 0.24 0.065 rpy=1.5708 -6.32034e-16 -3.14159
